File: hardware/butt_blaster_mk_2.sch (EAGLE design)
At the start: 23 parts, among them IC1 HV9922

Commit message: butts
Parts:
- removed B1: (no value), A_butts:RB1ANOSUCK
- removed CX1, CX2: 0.1uF, A_butts:CXXC10B5
- removed F1: 250mA(?), A_butts:FUSETR5
- removed IC1: HV9922, A_butts:HV9922
- removed JP1: M025MM, A_butts:M025MM
- removed L1: 10mH, A_butts:INDUCTORRLB0912
- removed L2: 10mH, A_butts:INDUCTORAXIAL-PTH-10.16MM
- removed LED7, LED8, LED9: LED5MM_SHORTPADS, A_butts:LED5MM_SHORTPADS
- removed MOV1: (no value), A_butts:VARISITORVAR-5.08MM-PTH
- added 12V: (no value), A_butts:DCBARRELPTH
- added Q1: 2N3904, A_butts:TRANSISTOR_NPNTO-92-AMMO-EBC
- added Q2: 2N7000, A_butts:MOSFET-NCHANNEL2N7000-AMMO
- added R1: 10R, A_butts:RESISTORPTH-AXIAL-7.68MM
- added R2: 10k, A_butts:RESISTORPTH-AXIAL-7.68MM
- added TVS1: (no value), A_butts:TVSDO-41-TVS-BIDIRECTIONAL
- C2: device A_butts:CAPACITOR-CERAMIC025-024X044 -> A_butts:CAPACITOR-POLARIZEDE2.5-6
- D1: device A_butts:DIODE-SCHOTTKYPTH-7.68MM -> A_butts:DIODE-SCHOTTKYPTH-8.38MM
Connections:
- removed net AC(L): F1.1, JP1.2
- removed net AC(N): B1.AC2, JP1.1, MOV1.P$1
- removed net N$10 (its old number): D1.A, IC1.DRAIN, L1.1
- removed net N$11: C2.1, CX2.1, D1.C, L2.2, LED1.A
- removed net N$13: B1.+, CX1.1, L2.1
- removed net N$14: C1.1, IC1.VDD
- removed net N$9: C2.2, L1.2, LED9.C
- new net VCC: C1.1, C2.+, D1.C, LED1.A, Q1.C, R2.1
- net GND: now also 12V.BRK, 12V.GND, C2.-, Q1.E, R1.2, TVS1.1; no longer B1.-, CX1.2, CX2.2, IC1.GND
- net N$12: now also 12V.PWR, D1.A, TVS1.2; no longer B1.AC1, F1.2, MOV1.P$2
- net N$6: now also Q1.B, Q2.S, R1.1; no longer LED6.C, LED7.A
- net N$7: now also LED6.C, Q2.D; no longer LED7.C, LED8.A
- net N$8: now also Q2.G, R2.2; no longer LED8.C, LED9.A
Other:
- moved on the sheet: C1, D1, LED1, LED2, LED3, LED4, LED5, LED6
