File: hardware/butt_blaster_mk_3.brd (EAGLE design)
At the start: 34 x 34 mm, 17 parts, among them Q1 2N3904, Q2 2N7000

Commit message: more butts, only twooooo leds this time
Parts:
- removed 12V: (no value), A_butts:DCJACK_2MM_PTH
- removed D1: 1N5819, A_butts:DIODE-10.16MM
- removed LED3, LED4, LED5, LED6: LED5MM_SHORTPADS, A_butts:LED5MM_SHORTPADS
- added D2: 10V, A_butts:DIODE-7.68MM
- added Q3: 2N3904, A_butts:TO-92-AMMO
- added Q4, Q5: 2N7000, A_butts:TO-92-AMMO
- added R3: 47R, A_butts:RESISTOR-AXIAL-PTH-7.68MM
- added R4, R5: 10k, A_butts:RESISTOR-AXIAL-PTH-6.35MM
- added U1: (no value), A_butts:USB-MICRO-B-FCI-CUTOUT
- LED2: value LED5MM_SHORTPADS -> LED3MM; device A_butts:LED5MM_SHORTPADS -> A_butts:LED3MM
- R2: device A_butts:RESISTOR-AXIAL-PTH-7.68MM -> A_butts:RESISTOR-AXIAL-PTH-6.35MM
- moved Q1 28.0 mm to (11.0, 24.5), turned to 270 degrees
- moved C1 21.6 mm to (11.0, 17.8), turned to 270 degrees
- moved Q2 20.5 mm to (17.0, 24.5), turned to 270 degrees
- moved TVS1 12.3 mm to (7.00, 19.0)
- moved R2 11.7 mm to (13.5, 21.2), turned to 90 degrees
- moved R1 10.3 mm to (17.0, 29.5)
- moved LED1 5.51 mm to (17.0, 18.0), turned to 90 degrees
- moved LED2 4.60 mm to (24.5, 11.2), turned to 90 degrees
- moved C2 3.13 mm to (41.8, 28.5), turned to 270 degrees
Connections:
- removed net N$10: LED5.K, LED6.A
- removed net N$12: 12V.PWR, D1.A, TVS1.P$2
- removed net N$7: LED6.K, Q2.3
- new net N$5: D2.K, Q5.2, R5.P$1
- new net N$9: D2.A, Q5.3, TVS1.P$1, U1.5, U1.P$1, U1.P$2
- net GND: now also Q3.1, Q5.1, R3.P$2; no longer 12V.BRK, 12V.GND, TVS1.P$1
- net N$1: now also LED1.K, Q2.3; no longer LED3.K, LED4.A
- net N$2: now also Q3.2, Q4.1, R3.P$1; no longer LED2.K, LED3.A
- net N$3: now also Q4.2, R4.P$2; no longer LED4.K, LED5.A
- net N$4: now also LED2.K, Q4.3; no longer LED1.K, LED2.A
- net VCC: now also LED2.A, Q3.3, R4.P$1, R5.P$2, TVS1.P$2, U1.1; no longer D1.C

Commit message: shuffled up componets but still not happy
Parts:
- R1, R3: device A_butts:RESISTOR-AXIAL-PTH-7.68MM -> A_butts:RESISTOR-AXIAL-PTH-10.16MM
- R4, R5: device A_butts:RESISTOR-AXIAL-PTH-6.35MM -> A_butts:RESISTOR-AXIAL-PTH-7.68MM
- moved C2 32.9 mm to (11.0, 16.8), turned to 180 degrees
- moved LED2 21.1 mm to (3.50, 9.75), turned to 0 degrees
- moved Q4 17.5 mm to (8.25, 24.5)
- moved R4 16.9 mm to (2.25, 20.8), turned to 90 degrees
- moved R2 16.8 mm to (30.2, 21.2)
- moved Q5 16.3 mm to (25.0, 10.8)
- moved TVS1 11.1 mm to (8.75, 8.00)
- moved Q3 10.5 mm to (14.0, 24.5), turned to 270 degrees
- moved Q1 8.75 mm to (19.8, 24.5)
- moved Q2 8.50 mm to (25.5, 24.5)
- moved C1 8.28 mm to (18.2, 13.8), turned to 0 degrees
- moved R1 2.50 mm to (17.0, 32.0), turned to 180 degrees
- moved R3 2.50 mm to (17.0, 29.5), turned to 0 degrees
- moved R5 0.50 mm to (17.0, 10.8), turned to 180 degrees
- moved D2 0.25 mm to (17.0, 7.75), turned to 0 degrees
Changed lines of the file:
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@@
 <setting verticaltext="up"/>
 </settings>
-<grid distance="0.25" unitdist="mm" unit="mm" style="lines" multiple="4" display="yes" altdistance="1" altunitdist="inch" altunit="inch"/>
+<grid distance="0.25" unitdist="mm" unit="mm" style="lines" multiple="4" display="yes" altdistance="1" altunitdist="mil" altunit="mil"/>
 <layers>
 <layer number="1" name="Top" color="4" fill="1" visible="yes" active="yes"/>
@@
 <element name="H2" library="A_butts" package="HOLE-#2" value="HOLE#2" x="27" y="2.75"/>
 <element name="LED1" library="A_butts" package="LED5MM_SHORTPADS" value="LED5MM_SHORTPADS" x="17" y="18" rot="R90"/>
-<element name="C1" library="A_butts" package="C025-024X044" value="0.1uF" x="11" y="17.75" rot="R270"/>
-<element name="C2" library="A_butts" package="E2,5-6" value="10uF" x="41.75" y="28.5" rot="R270"/>
-<element name="TVS1" library="A_butts" package="DO-41-TVS" value="" x="7" y="19" rot="R90"/>
-<element name="Q1" library="A_butts" package="TO-92-AMMO" value="2N3904" x="11" y="24.5" rot="R270"/>
-<element name="Q2" library="A_butts" package="TO-92-AMMO" value="2N7000" x="17" y="24.5" rot="R270"/>
-<element name="R1" library="A_butts" package="RESISTOR-AXIAL-PTH-7.68MM" value="10R" x="17" y="29.5"/>
-<element name="R2" library="A_butts" package="RESISTOR-AXIAL-PTH-6.35MM" value="10k" x="13.5" y="21.25" rot="R90"/>
+<element name="C1" library="A_butts" package="C025-024X044" value="0.1uF" x="18.25" y="13.75"/>
+<element name="C2" library="A_butts" package="E2,5-6" value="10uF" x="11" y="16.75" rot="R180"/>
+<element name="TVS1" library="A_butts" package="DO-41-TVS" value="" x="8.75" y="8" rot="R90"/>
+<element name="Q1" library="A_butts" package="TO-92-AMMO" value="2N3904" x="19.75" y="24.5" rot="R270"/>
+<element name="Q2" library="A_butts" package="TO-92-AMMO" value="2N7000" x="25.5" y="24.5" rot="R270"/>
+<element name="R1" library="A_butts" package="RESISTOR-AXIAL-PTH-10.16MM" value="10R" x="17" y="32" rot="R180"/>
+<element name="R2" library="A_butts" package="RESISTOR-AXIAL-PTH-6.35MM" value="10k" x="30.25" y="21.25" rot="R90"/>
 <element name="U1" library="A_butts" package="USB-MICRO-B-FCI-CUTOUT" value="" x="17" y="5"/>
-<element name="LED2" library="A_butts" package="LED3MM" value="LED3MM" x="24.5" y="11.25" rot="R90"/>
-<element name="Q3" library="A_butts" package="TO-92-AMMO" value="2N3904" x="24.5" y="24.75" rot="R180"/>
-<element name="Q4" library="A_butts" package="TO-92-AMMO" value="2N7000" x="24.5" y="18" rot="R270"/>
-<element name="R3" library="A_butts" package="RESISTOR-AXIAL-PTH-7.68MM" value="47R" x="17" y="32" rot="R180"/>
-<element name="R4" library="A_butts" package="RESISTOR-AXIAL-PTH-6.35MM" value="10k" x="17" y="12.5"/>
-<element name="Q5" library="A_butts" package="TO-92-AMMO" value="2N7000" x="8.75" y="10.25" rot="R270"/>
-<element name="D2" library="A_butts" package="DIODE-7.68MM" value="10V" x="17" y="7.5" rot="R180"/>
-<element name="R5" library="A_butts" package="RESISTOR-AXIAL-PTH-6.35MM" value="10k" x="17" y="10.25"/>
+<element name="LED2" library="A_butts" package="LED3MM" value="LED3MM" x="3.5" y="9.75"/>
+<element name="Q3" library="A_butts" package="TO-92-AMMO" value="2N3904" x="14" y="24.5" rot="R270"/>
+<element name="Q4" library="A_butts" package="TO-92-AMMO" value="2N7000" x="8.25" y="24.5" rot="R270"/>
+<element name="R3" library="A_butts" package="RESISTOR-AXIAL-PTH-10.16MM" value="47R" x="17" y="29.5"/>
+<element name="R4" library="A_butts" package="RESISTOR-AXIAL-PTH-7.68MM" value="10k" x="2.25" y="20.75" rot="R90"/>
+<element name="Q5" library="A_butts" package="TO-92-AMMO" value="2N7000" x="25" y="10.75" rot="R270"/>
+<element name="D2" library="A_butts" package="DIODE-7.68MM" value="10V" x="17" y="7.75"/>
+<element name="R5" library="A_butts" package="RESISTOR-AXIAL-PTH-7.68MM" value="10k" x="17" y="10.75" rot="R180"/>
 </elements>
 <signals>
@@
 <contactref element="R1" pad="P$1"/>
 <contactref element="Q1" pad="2"/>
-<wire x1="13.19" y1="29.5" x2="17" y2="27.04" width="0" layer="19" extent="1-1"/>
-<wire x1="11" y1="24.5" x2="13.19" y2="29.5" width="0" layer="19" extent="1-1"/>
+<wire x1="22.08" y1="32" x2="25.5" y2="27.04" width="0" layer="19" extent="1-1"/>
+<wire x1="19.75" y1="24.5" x2="25.5" y2="27.04" width="0" layer="19" extent="1-1"/>
 </signal>
 <signal name="GND">
@@
 </polygon>
 <contactref element="Q5" pad="1"/>
-<wire x1="27.04" y1="24.75" x2="41.75" y2="27.23" width="0" layer="19" extent="1-1"/>
 </signal>
 <signal name="N$8">
 <contactref element="Q2" pad="2"/>
 <contactref element="R2" pad="P$2"/>
-<wire x1="13.5" y1="24.425" x2="17" y2="24.5" width="0" layer="19" extent="1-1"/>
+<wire x1="25.5" y1="24.5" x2="30.25" y2="24.425" width="0" layer="19" extent="1-1"/>
 </signal>
 <signal name="VCC">
@@
 <contactref element="R5" pad="P$2"/>
 <contactref element="TVS1" pad="P$2"/>
-<wire x1="21.96" y1="24.75" x2="41.75" y2="29.77" width="0" layer="19" extent="1-1"/>
-<wire x1="17" y1="16.73" x2="21.96" y2="24.75" width="0" layer="19" extent="1-1"/>
-<wire x1="13.5" y1="18.075" x2="17" y2="16.73" width="0" layer="19" extent="1-1"/>
-<wire x1="11" y1="19.02" x2="13.5" y2="18.075" width="0" layer="19" extent="1-1"/>
-<wire x1="13.825" y1="12.5" x2="17" y2="16.73" width="0" layer="19" extent="1-1"/>
-<wire x1="11" y1="21.96" x2="11" y2="19.02" width="0" layer="19" extent="1-1"/>
-<wire x1="7" y1="24.08" x2="11" y2="21.96" width="0" layer="19" extent="1-1"/>
-<wire x1="20.175" y1="10.25" x2="13.825" y2="12.5" width="0" layer="19" extent="1-1"/>
-<wire x1="24.5" y1="9.98" x2="20.175" y2="10.25" width="0" layer="19" extent="1-1"/>
-<wire x1="15.7" y1="5" x2="20.175" y2="10.25" width="0" layer="19" extent="1-1"/>
+<wire x1="19.75" y1="21.96" x2="30.25" y2="18.075" width="0" layer="19" extent="1-1"/>
+<wire x1="14" y1="21.96" x2="19.75" y2="21.96" width="0" layer="19" extent="1-1"/>
+<wire x1="12.27" y1="16.75" x2="14" y2="21.96" width="0" layer="19" extent="1-1"/>
+<wire x1="17" y1="16.73" x2="12.27" y2="16.75" width="0" layer="19" extent="1-1"/>
+<wire x1="16.98" y1="13.75" x2="17" y2="16.73" width="0" layer="19" extent="1-1"/>
+<wire x1="13.19" y1="10.75" x2="16.98" y2="13.75" width="0" layer="19" extent="1-1"/>
+<wire x1="8.75" y1="13.08" x2="13.19" y2="10.75" width="0" layer="19" extent="1-1"/>
+<wire x1="15.7" y1="5" x2="13.19" y2="10.75" width="0" layer="19" extent="1-1"/>
+<wire x1="2.23" y1="9.75" x2="8.75" y2="13.08" width="0" layer="19" extent="1-1"/>
+<wire x1="2.25" y1="16.94" x2="2.23" y2="9.75" width="0" layer="19" extent="1-1"/>
 </signal>
 <signal name="N$1">
 <contactref element="Q2" pad="3"/>
 <contactref element="LED1" pad="K"/>
-<wire x1="17" y1="19.27" x2="17" y2="21.96" width="0" layer="19" extent="1-1"/>
+<wire x1="17" y1="19.27" x2="25.5" y2="21.96" width="0" layer="19" extent="1-1"/>
 </signal>
 <signal name="N$2">
@@
 <contactref element="R3" pad="P$1"/>
 <contactref element="Q3" pad="2"/>
-<wire x1="24.5" y1="24.75" x2="20.81" y2="32" width="0" layer="19" extent="1-1"/>
-<wire x1="24.5" y1="20.54" x2="24.5" y2="24.75" width="0" layer="19" extent="1-1"/>
+<wire x1="8.25" y1="27.04" x2="11.92" y2="29.5" width="0" layer="19" extent="1-1"/>
+<wire x1="14" y1="24.5" x2="11.92" y2="29.5" width="0" layer="19" extent="1-1"/>
 </signal>
 <signal name="N$3">
 <contactref element="Q4" pad="2"/>
 <contactref element="R4" pad="P$2"/>
-<wire x1="20.175" y1="12.5" x2="24.5" y2="18" width="0" layer="19" extent="1-1"/>
+<wire x1="2.25" y1="24.56" x2="8.25" y2="24.5" width="0" layer="19" extent="1-1"/>
 </signal>
 <signal name="N$4">
 <contactref element="Q4" pad="3"/>
 <contactref element="LED2" pad="K"/>
-<wire x1="24.5" y1="12.52" x2="24.5" y2="15.46" width="0" layer="19" extent="1-1"/>
+<wire x1="4.77" y1="9.75" x2="8.25" y2="21.96" width="0" layer="19" extent="1-1"/>
 </signal>
 <signal name="N$5">
@@
 <contactref element="R5" pad="P$1"/>
 <contactref element="D2" pad="K"/>
-<wire x1="13.19" y1="7.5" x2="13.825" y2="10.25" width="0" layer="19" extent="1-1"/>
-<wire x1="8.75" y1="10.25" x2="13.825" y2="10.25" width="0" layer="19" extent="1-1"/>
+<wire x1="20.81" y1="10.75" x2="25" y2="10.75" width="0" layer="19" extent="1-1"/>
+<wire x1="20.81" y1="7.75" x2="20.81" y2="10.75" width="0" layer="19" extent="1-1"/>
 </signal>
 <signal name="N$9">
@@
 <contactref element="U1" pad="P$2"/>
 <contactref element="TVS1" pad="P$1"/>
-<wire x1="19.325" y1="5" x2="20.81" y2="7.5" width="0" layer="19" extent="1-1"/>
+<wire x1="19.325" y1="5" x2="25" y2="8.21" width="0" layer="19" extent="1-1"/>
 <wire x1="18.3" y1="5" x2="19.325" y2="5" width="0" layer="19" extent="1-1"/>
 <wire x1="14.675" y1="5" x2="18.3" y2="5" width="0" layer="19" extent="1-1"/>
-<wire x1="8.75" y1="7.71" x2="14.675" y2="5" width="0" layer="19" extent="1-1"/>
-<wire x1="7" y1="13.92" x2="8.75" y2="7.71" width="0" layer="19" extent="1-1"/>
+<wire x1="13.19" y1="7.75" x2="14.675" y2="5" width="0" layer="19" extent="1-1"/>
+<wire x1="8.75" y1="2.92" x2="14.675" y2="5" width="0" layer="19" extent="1-1"/>
 </signal>
 </signals>

Commit message: huh
Parts:
- removed Q3: 2N3904, A_butts:TO-92-AMMO
- removed Q4: 2N7000, A_butts:TO-92-AMMO
- removed R4: 10k, A_butts:RESISTOR-AXIAL-PTH-7.68MM
- removed U1: (no value), A_butts:USB-MICRO-B-FCI-CUTOUT
- added F1: 250mA, A_butts:PTC
- added LED3: LED3MM, A_butts:LED3MM
- added PWR: (no value), A_butts:USB-MICRO-B-FCI-CUTOUT
- added U$2: (no value), A_butts:COW_SMALL
- added U$3, U$4: (no value), A_butts:CC-BY-SA-4.0-NO-URL
- added U$5: (no value), A_butts:OSHWLOGO_TOP_0.2_A
- LED2: value LED3MM -> LED5MM_SHORTPADS; device A_butts:LED3MM -> A_butts:LED5MM_SHORTPADS
- R3: value 47R -> 1k; device A_butts:RESISTOR-AXIAL-PTH-10.16MM -> A_butts:RESISTOR-AXIAL-PTH-6.35MM
- moved LED2 14.8 mm to (15.8, 18.0), turned to 90 degrees
- moved C1 13.5 mm to (7.00, 21.3), turned to 270 degrees
- moved R3 13.0 mm to (5.00, 24.4), turned to 270 degrees
- moved R2 9.77 mm to (20.5, 21.8)
- moved Q2 9.76 mm to (15.8, 25.0)
- moved Q1 9.51 mm to (10.2, 25.0)
- moved C2 7.27 mm to (3.73, 16.7)
- moved LED1 6.75 mm to (10.2, 18.0)
- moved Q5 4.51 mm to (20.5, 11.0)
- moved D2 4.07 mm to (13.0, 8.50)
- moved R5 4.01 mm to (13.0, 11.0)
- moved H1 4.00 mm to (3.00, 31.2)
- moved H2 4.00 mm to (23.0, 2.75)
- moved TVS1 3.79 mm to (5.00, 7.42)
- moved R1 1.25 mm to (16.0, 31.2), turned to 0 degrees
Connections:
- removed net N$9: D2.A, Q5.3, TVS1.P$1, U1.5, U1.P$1, U1.P$2
- new net REAL_GND: D2.A, PWR.5, PWR.P$1, PWR.P$2, Q5.3, TVS1.P$1
- net GND: now also LED3.K; no longer Q3.1, R3.P$2
- net N$1: now also LED2.A; no longer Q2.3
- net N$2: now also LED3.A; no longer Q3.2, Q4.1
- net N$3: now also LED2.K, Q2.3; no longer Q4.2, R4.P$2
- net N$4: now also F1.P$1, PWR.1; no longer LED2.K, Q4.3
- net VCC: now also F1.P$2, R3.P$2; no longer LED2.A, Q3.3, R4.P$1, U1.1
Routing:
- net VCC: track 0.00 -> 36.7 mm
- net N$6: track 0.00 -> 12.9 mm
- net N$4: track 0.00 -> 8.29 mm
- net N$1: track 0.00 -> 6.55 mm
- net N$5: track 0.00 -> 6.19 mm
- net N$8: track 0.00 -> 4.76 mm
- net N$2: track 0.00 -> 3.37 mm
- net N$3: track 0.00 -> 3.19 mm
- added copper zone on layer 16, net REAL_GND
Other:
- board size 34 x 34 mm -> 26 x 34 mm
