File: hardware/butt_blaster_mk_3.sch (EAGLE design)
At the start: 17 parts, among them Q1 2N3904, Q2 2N7000

Commit message: more butts, only twooooo leds this time
Parts:
- removed 12V: (no value), A_butts:DCBARRELPTH
- removed D1: 1N5819, A_butts:DIODE-SCHOTTKYPTH-10.16MM
- removed LED3, LED4, LED5, LED6: LED5MM_SHORTPADS, A_butts:LED5MM_SHORTPADS
- added D2: 10V, A_butts:DIODE-ZENERPTH-7.68MM
- added Q3: 2N3904, A_butts:TRANSISTOR_NPNTO-92-AMMO-EBC
- added Q4, Q5: 2N7000, A_butts:MOSFET-NCHANNEL2N7000-AMMO
- added R3: 47R, A_butts:RESISTORPTH-AXIAL-7.68MM
- added R4, R5: 10k, A_butts:RESISTORPTH-AXIAL-6.35MM
- added U1: (no value), A_butts:USB-ABCOMBO
- LED2: value LED5MM_SHORTPADS -> LED3MM; device A_butts:LED5MM_SHORTPADS -> A_butts:LED3MM
- R2: device A_butts:RESISTORPTH-AXIAL-7.68MM -> A_butts:RESISTORPTH-AXIAL-6.35MM
Connections:
- removed net N$10: LED5.C, LED6.A
- removed net N$12: 12V.PWR, D1.A, TVS1.2
- removed net N$7: LED6.C, Q2.D
- new net N$5: D2.C, Q5.G, R5.1
- new net N$9: D2.A, Q5.D, TVS1.1, U1.GND
- net GND: now also Q3.E, Q5.S, R3.2; no longer 12V.BRK, 12V.GND, TVS1.1
- net N$1: now also LED1.C, Q2.D; no longer LED3.C, LED4.A
- net N$2: now also Q3.B, Q4.S, R3.1; no longer LED2.C, LED3.A
- net N$3: now also Q4.G, R4.2; no longer LED4.C, LED5.A
- net N$4: now also LED2.C, Q4.D; no longer LED1.C, LED2.A
- net VCC: now also LED2.A, Q3.C, R4.1, R5.2, TVS1.2, U1.VBUS; no longer D1.C
Other:
- moved on the sheet: C1, C2, LED1, LED2, Q1, Q2, R1, R2, TVS1

Commit message: shuffled up componets but still not happy
Parts:
- R1, R3: device A_butts:RESISTORPTH-AXIAL-7.68MM -> A_butts:RESISTORPTH-AXIAL-10.16MM
- R4, R5: device A_butts:RESISTORPTH-AXIAL-6.35MM -> A_butts:RESISTORPTH-AXIAL-7.68MM
Changed lines of the file:
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@@
 <setting verticaltext="up"/>
 </settings>
-<grid distance="100" unitdist="mil" unit="mil" style="lines" multiple="1" display="yes" altdistance="1" altunitdist="mil" altunit="mil"/>
+<grid distance="100" unitdist="mil" unit="mil" style="lines" multiple="1" display="yes" altdistance="2" altunitdist="mil" altunit="mil"/>
 <layers>
 <layer number="1" name="Top" color="4" fill="1" visible="yes" active="no"/>
@@
 <part name="Q1" library="A_butts" deviceset="TRANSISTOR_NPN" device="TO-92-AMMO-EBC" value="2N3904"/>
 <part name="Q2" library="A_butts" deviceset="MOSFET-NCHANNEL" device="2N7000-AMMO" value="2N7000"/>
-<part name="R1" library="A_butts" deviceset="RESISTOR" device="PTH-AXIAL-7.68MM" value="10R"/>
+<part name="R1" library="A_butts" deviceset="RESISTOR" device="PTH-AXIAL-10.16MM" value="10R"/>
 <part name="R2" library="A_butts" deviceset="RESISTOR" device="PTH-AXIAL-6.35MM" value="10k"/>
 <part name="GND1" library="A_butts" deviceset="GND" device=""/>
@@
 <part name="Q3" library="A_butts" deviceset="TRANSISTOR_NPN" device="TO-92-AMMO-EBC" value="2N3904"/>
 <part name="Q4" library="A_butts" deviceset="MOSFET-NCHANNEL" device="2N7000-AMMO" value="2N7000"/>
-<part name="R3" library="A_butts" deviceset="RESISTOR" device="PTH-AXIAL-7.68MM" value="47R"/>
-<part name="R4" library="A_butts" deviceset="RESISTOR" device="PTH-AXIAL-6.35MM" value="10k"/>
+<part name="R3" library="A_butts" deviceset="RESISTOR" device="PTH-AXIAL-10.16MM" value="47R"/>
+<part name="R4" library="A_butts" deviceset="RESISTOR" device="PTH-AXIAL-7.68MM" value="10k"/>
 <part name="SUPPLY3" library="A_butts" deviceset="VCC" device=""/>
 <part name="Q5" library="A_butts" deviceset="MOSFET-NCHANNEL" device="2N7000-AMMO" value="2N7000"/>
 <part name="D2" library="A_butts" deviceset="DIODE-ZENER" device="PTH-7.68MM" value="10V"/>
-<part name="R5" library="A_butts" deviceset="RESISTOR" device="PTH-AXIAL-6.35MM" value="10k"/>
+<part name="R5" library="A_butts" deviceset="RESISTOR" device="PTH-AXIAL-7.68MM" value="10k"/>
 </parts>
 <sheets>

Commit message: huh
Parts:
- removed Q3: 2N3904, A_butts:TRANSISTOR_NPNTO-92-AMMO-EBC
- removed Q4: 2N7000, A_butts:MOSFET-NCHANNEL2N7000-AMMO
- removed R4: 10k, A_butts:RESISTORPTH-AXIAL-7.68MM
- removed U1: (no value), A_butts:USB-ABCOMBO
- added F1: 250mA, A_butts:PTCPTH
- added LED3: LED3MM, A_butts:LED3MM
- added PWR: (no value), A_butts:USB-ABCOMBO
- LED2: value LED3MM -> LED5MM_SHORTPADS; device A_butts:LED3MM -> A_butts:LED5MM_SHORTPADS
- R3: value 47R -> 1k; device A_butts:RESISTORPTH-AXIAL-10.16MM -> A_butts:RESISTORPTH-AXIAL-6.35MM
Connections:
- removed net N$9: D2.A, Q5.D, TVS1.1, U1.GND
- new net REAL_GND: D2.A, PWR.GND, Q5.D, TVS1.1
- net GND: now also LED3.C; no longer Q3.E, R3.2
- net N$1: now also LED2.A; no longer Q2.D
- net N$2: now also LED3.A; no longer Q3.B, Q4.S
- net N$3: now also LED2.C, Q2.D; no longer Q4.G, R4.2
- net N$4: now also F1.1, PWR.VBUS; no longer LED2.C, Q4.D
- net VCC: now also F1.2, R3.2; no longer LED2.A, Q3.C, R4.1, U1.VBUS
Other:
- moved on the sheet: LED1, LED2, R3
Changed lines of the file:
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@@
 <part name="R2" library="A_butts" deviceset="RESISTOR" device="PTH-AXIAL-6.35MM" value="10k"/>
 <part name="GND1" library="A_butts" deviceset="GND" device=""/>
-<part name="U1" library="A_butts" deviceset="USB-AB" device="COMBO"/>
+<part name="PWR" library="A_butts" deviceset="USB-AB" device="COMBO"/>
 <part name="SUPPLY2" library="A_butts" deviceset="VCC" device=""/>
-<part name="LED2" library="A_butts" deviceset="LED" device="3MM" value="LED3MM"/>
-<part name="GND2" library="A_butts" deviceset="GND" device=""/>
-<part name="Q3" library="A_butts" deviceset="TRANSISTOR_NPN" device="TO-92-AMMO-EBC" value="2N3904"/>
-<part name="Q4" library="A_butts" deviceset="MOSFET-NCHANNEL" device="2N7000-AMMO" value="2N7000"/>
-<part name="R3" library="A_butts" deviceset="RESISTOR" device="PTH-AXIAL-10.16MM" value="47R"/>
-<part name="R4" library="A_butts" deviceset="RESISTOR" device="PTH-AXIAL-7.68MM" value="10k"/>
-<part name="SUPPLY3" library="A_butts" deviceset="VCC" device=""/>
+<part name="R3" library="A_butts" deviceset="RESISTOR" device="PTH-AXIAL-6.35MM" value="1k"/>
 <part name="Q5" library="A_butts" deviceset="MOSFET-NCHANNEL" device="2N7000-AMMO" value="2N7000"/>
 <part name="D2" library="A_butts" deviceset="DIODE-ZENER" device="PTH-7.68MM" value="10V"/>
 <part name="R5" library="A_butts" deviceset="RESISTOR" device="PTH-AXIAL-7.68MM" value="10k"/>
+<part name="LED3" library="A_butts" deviceset="LED" device="3MM" value="LED3MM"/>
+<part name="LED2" library="A_butts" deviceset="LED" device="5MM_SHORTPADS"/>
+<part name="F1" library="A_butts" deviceset="PTC" device="PTH" value="250mA"/>
 </parts>
 <sheets>
@@
 <instance part="H1" gate="G$1" x="106.68" y="63.5"/>
 <instance part="H2" gate="G$1" x="111.76" y="63.5"/>
-<instance part="LED1" gate="G$1" x="35.56" y="96.52" rot="MR0"/>
+<instance part="LED1" gate="G$1" x="20.32" y="101.6" rot="MR270"/>
 <instance part="C1" gate="G$1" x="50.8" y="25.4"/>
 <instance part="GND3" gate="1" x="22.86" y="55.88"/>
@@
 <instance part="R2" gate="G$1" x="20.32" y="83.82"/>
 <instance part="GND1" gate="1" x="60.96" y="7.62"/>
-<instance part="U1" gate="G$1" x="15.24" y="33.02"/>
-<instance part="SUPPLY2" gate="G$1" x="22.86" y="104.14"/>
-<instance part="LED2" gate="G$1" x="81.28" y="96.52" rot="MR0"/>
-<instance part="GND2" gate="1" x="68.58" y="55.88"/>
-<instance part="Q3" gate="G$1" x="58.42" y="76.2" rot="MR0"/>
-<instance part="Q4" gate="G$1" x="81.28" y="83.82"/>
-<instance part="R3" gate="G$1" x="81.28" y="68.58" rot="R270"/>
-<instance part="R4" gate="G$1" x="66.04" y="83.82"/>
-<instance part="SUPPLY3" gate="G$1" x="68.58" y="104.14"/>
+<instance part="PWR" gate="G$1" x="7.62" y="33.02"/>
+<instance part="SUPPLY2" gate="G$1" x="10.16" y="104.14"/>
+<instance part="R3" gate="G$1" x="71.12" y="30.48" rot="R90"/>
 <instance part="Q5" gate="G$1" x="43.18" y="12.7" rot="MR270"/>
 <instance part="D2" gate="G$1" x="35.56" y="17.78" rot="R90"/>
 <instance part="R5" gate="G$1" x="43.18" y="30.48" rot="R90"/>
+<instance part="LED3" gate="G$1" x="71.12" y="20.32"/>
+<instance part="LED2" gate="G$1" x="35.56" y="96.52" rot="MR0"/>
+<instance part="F1" gate="G$1" x="17.78" y="38.1"/>
 </instances>
 <busses>
@@
 <wire x1="48.26" y1="12.7" x2="50.8" y2="12.7" width="0.1524" layer="91"/>
 <pinref part="Q5" gate="G$1" pin="S"/>
-</segment>
-<segment>
-<pinref part="R3" gate="G$1" pin="2"/>
-<pinref part="GND2" gate="1" pin="GND"/>
-<wire x1="68.58" y1="58.42" x2="68.58" y2="60.96" width="0.1524" layer="91"/>
-<wire x1="68.58" y1="60.96" x2="81.28" y2="60.96" width="0.1524" layer="91"/>
-<wire x1="81.28" y1="60.96" x2="81.28" y2="63.5" width="0.1524" layer="91"/>
-<pinref part="Q3" gate="G$1" pin="E"/>
-<wire x1="55.88" y1="71.12" x2="55.88" y2="60.96" width="0.1524" layer="91"/>
-<wire x1="55.88" y1="60.96" x2="68.58" y2="60.96" width="0.1524" layer="91"/>
-<junction x="68.58" y="60.96"/>
+<wire x1="60.96" y1="12.7" x2="71.12" y2="12.7" width="0.1524" layer="91"/>
+<wire x1="71.12" y1="12.7" x2="71.12" y2="15.24" width="0.1524" layer="91"/>
+<pinref part="LED3" gate="G$1" pin="C"/>
 </segment>
 </net>
@@
 <wire x1="50.8" y1="38.1" x2="60.96" y2="38.1" width="0.1524" layer="91"/>
 <wire x1="50.8" y1="38.1" x2="50.8" y2="30.48" width="0.1524" layer="91"/>
-<pinref part="U1" gate="G$1" pin="VBUS"/>
-<wire x1="17.78" y1="38.1" x2="27.94" y2="38.1" width="0.1524" layer="91"/>
 <pinref part="R5" gate="G$1" pin="2"/>
 <wire x1="27.94" y1="38.1" x2="43.18" y2="38.1" width="0.1524" layer="91"/>
@@
 <pinref part="TVS1" gate="G$1" pin="2"/>
 <wire x1="27.94" y1="33.02" x2="27.94" y2="38.1" width="0.1524" layer="91"/>
-<junction x="27.94" y="38.1"/>
 <wire x1="43.18" y1="38.1" x2="50.8" y2="38.1" width="0.1524" layer="91"/>
 <junction x="43.18" y="38.1"/>
 <junction x="50.8" y="38.1"/>
+<wire x1="60.96" y1="38.1" x2="71.12" y2="38.1" width="0.1524" layer="91"/>
+<pinref part="R3" gate="G$1" pin="2"/>
+<wire x1="71.12" y1="38.1" x2="71.12" y2="35.56" width="0.1524" layer="91"/>
+<pinref part="F1" gate="G$1" pin="2"/>
+<wire x1="25.4" y1="38.1" x2="27.94" y2="38.1" width="0.1524" layer="91"/>
+<junction x="27.94" y="38.1"/>
 </segment>
 <segment>
@@
 <junction x="10.16" y="83.82"/>
 <pinref part="LED1" gate="G$1" pin="A"/>
-<wire x1="35.56" y1="99.06" x2="35.56" y2="101.6" width="0.1524" layer="91"/>
-<wire x1="35.56" y1="101.6" x2="22.86" y2="101.6" width="0.1524" layer="91"/>
-<wire x1="22.86" y1="101.6" x2="10.16" y2="101.6" width="0.1524" layer="91"/>
+<wire x1="17.78" y1="101.6" x2="10.16" y2="101.6" width="0.1524" layer="91"/>
 <wire x1="10.16" y1="101.6" x2="10.16" y2="83.82" width="0.1524" layer="91"/>
 <junction x="10.16" y="83.82"/>
 <pinref part="SUPPLY2" gate="G$1" pin="VCC"/>
-<wire x1="22.86" y1="101.6" x2="22.86" y2="104.14" width="0.1524" layer="91"/>
-<junction x="22.86" y="101.6"/>
-</segment>
-<segment>
-<pinref part="Q3" gate="G$1" pin="C"/>
-<wire x1="55.88" y1="81.28" x2="55.88" y2="83.82" width="0.1524" layer="91"/>
-<pinref part="R4" gate="G$1" pin="1"/>
-<wire x1="55.88" y1="83.82" x2="60.96" y2="83.82" width="0.1524" layer="91"/>
-<junction x="55.88" y="83.82"/>
-<pinref part="LED2" gate="G$1" pin="A"/>
-<wire x1="81.28" y1="99.06" x2="81.28" y2="101.6" width="0.1524" layer="91"/>
-<wire x1="81.28" y1="101.6" x2="68.58" y2="101.6" width="0.1524" layer="91"/>
-<wire x1="68.58" y1="101.6" x2="55.88" y2="101.6" width="0.1524" layer="91"/>
-<wire x1="55.88" y1="101.6" x2="55.88" y2="83.82" width="0.1524" layer="91"/>
-<junction x="55.88" y="83.82"/>
-<pinref part="SUPPLY3" gate="G$1" pin="VCC"/>
-<wire x1="68.58" y1="101.6" x2="68.58" y2="104.14" width="0.1524" layer="91"/>
-<junction x="68.58" y="101.6"/>
-</segment>
-</net>
-<net name="N$1" class="0">
-<segment>
-<pinref part="Q2" gate="G$1" pin="D"/>
-<pinref part="LED1" gate="G$1" pin="C"/>
-<wire x1="35.56" y1="91.44" x2="35.56" y2="88.9" width="0.1524" layer="91"/>
-</segment>
-</net>
-<net name="N$2" class="0">
-<segment>
-<pinref part="Q4" gate="G$1" pin="S"/>
-<pinref part="R3" gate="G$1" pin="1"/>
-<wire x1="81.28" y1="73.66" x2="81.28" y2="76.2" width="0.1524" layer="91"/>
-<pinref part="Q3" gate="G$1" pin="B"/>
-<wire x1="81.28" y1="76.2" x2="81.28" y2="78.74" width="0.1524" layer="91"/>
-<wire x1="60.96" y1="76.2" x2="81.28" y2="76.2" width="0.1524" layer="91"/>
-<junction x="81.28" y="76.2"/>
-</segment>
-</net>
-<net name="N$3" class="0">
-<segment>
-<pinref part="Q4" gate="G$1" pin="G"/>
-<pinref part="R4" gate="G$1" pin="2"/>
-<wire x1="71.12" y1="83.82" x2="73.66" y2="83.82" width="0.1524" layer="91"/>
-</segment>
-</net>
-<net name="N$4" class="0">
-<segment>
-<pinref part="Q4" gate="G$1" pin="D"/>
-<pinref part="LED2" gate="G$1" pin="C"/>
-<wire x1="81.28" y1="91.44" x2="81.28" y2="88.9" width="0.1524" layer="91"/>
+<wire x1="10.16" y1="101.6" x2="10.16" y2="104.14" width="0.1524" layer="91"/>
+<junction x="10.16" y="101.6"/>
 </segment>
 </net>
@@
 </segment>
 </net>
-<net name="N$9" class="0">
+<net name="REAL_GND" class="0">
 <segment>
 <pinref part="Q5" gate="G$1" pin="D"/>
@@
 <wire x1="27.94" y1="12.7" x2="20.32" y2="12.7" width="0.1524" layer="91"/>
 <wire x1="20.32" y1="12.7" x2="20.32" y2="27.94" width="0.1524" layer="91"/>
-<pinref part="U1" gate="G$1" pin="GND"/>
-<wire x1="20.32" y1="27.94" x2="17.78" y2="27.94" width="0.1524" layer="91"/>
+<pinref part="PWR" gate="G$1" pin="GND"/>
+<wire x1="20.32" y1="27.94" x2="10.16" y2="27.94" width="0.1524" layer="91"/>
 <pinref part="TVS1" gate="G$1" pin="1"/>
 <wire x1="27.94" y1="22.86" x2="27.94" y2="12.7" width="0.1524" layer="91"/>
 <junction x="27.94" y="12.7"/>
+<label x="15.24" y="15.24" size="1.27" layer="95"/>
 </segment>
 </net>
+<net name="N$2" class="0">
+<segment>
+<pinref part="R3" gate="G$1" pin="1"/>
+<wire x1="71.12" y1="22.86" x2="71.12" y2="25.4" width="0.1524" layer="91"/>
+<pinref part="LED3" gate="G$1" pin="A"/>
+</segment>
+</net>
+<net name="N$1" class="0">
+<segment>
+<pinref part="LED1" gate="G$1" pin="C"/>
+<pinref part="LED2" gate="G$1" pin="A"/>
+<wire x1="35.56" y1="99.06" x2="35.56" y2="101.6" width="0.1524" layer="91"/>
+<wire x1="35.56" y1="101.6" x2="25.4" y2="101.6" width="0.1524" layer="91"/>
+</segment>
+</net>
+<net name="N$3" class="0">
+<segment>
+<pinref part="Q2" gate="G$1" pin="D"/>
+<pinref part="LED2" gate="G$1" pin="C"/>
+<wire x1="35.56" y1="91.44" x2="35.56" y2="88.9" width="0.1524" layer="91"/>
+</segment>
+</net>
+<net name="N$4" class="0">
+<segment>
+<pinref part="PWR" gate="G$1" pin="VBUS"/>
+<pinref part="F1" gate="G$1" pin="1"/>
+<wire x1="12.7" y1="38.1" x2="10.16" y2="38.1" width="0.1524" layer="91"/>
+</segment>
+</net>
